Commit message: add position control

File: simple_dog_simulation/simpledog/urdf/laikago/my_laika.xacro (robot description, xacro)
@@ -106,4 +106,20 @@
         </collision>
     </link>
+    <xacro:include filename="$(find simpledog)/urdf/front_kinect.urdf.xacro"/>
+    <xacro:include filename="$(find simpledog)/urdf/right_kinect.urdf.xacro"/>
+    <!--load kinect urdf-->
+      <xacro:front_kinect_camera prefix="front_camera" robot_namespace="$(arg robot_namespace)"/>
+      <joint name="front_kinect_frame_joint" type="fixed">
+        <origin xyz="0.28 0 0.0" rpy="0 0.8 0" />
+        <parent link="base"/>
+        <child link="front_camera_link"/>
+      </joint>
+    <!--load kinect urdf-->
+      <xacro:right_kinect_camera prefix="right_camera" robot_namespace="$(arg robot_namespace)"/>
+      <joint name="right_kinect_frame_joint" type="fixed">
+        <origin xyz="-0.0 -0.07 0.0" rpy="0 0.8 -1.57" />
+        <parent link="base"/>
+        <child link="right_camera_link"/>
+      </joint>
     <xacro:leg name="LF" mirror="1" mirror_dae="true" front_hind="1" front_hind_dae="true">
         <origin rpy="0 0 0" xyz="${leg_offset_x} ${leg_offset_y} 0"/>

File: simple_dog_simulation/simpledog/urdf/right_kinect.urdf.xacro (robot description, xacro)
@@ -25,6 +25,6 @@
 SOFTWARE, EVEN IF ADVISED OF THE POSSIBILITY OF SUCH DAMAGE.
 -->
-<robot xmlns:xacro="http://ros.org/wiki/xacro" name="kinect_camera">
-  <xacro:macro name="kinect_camera" params="prefix:=camera robot_namespace:=/">
+<robot xmlns:xacro="http://ros.org/wiki/xacro" name="right_kinect_camera">
+  <xacro:macro name="right_kinect_camera" params="prefix:=right_camera robot_namespace:=/">
     <!-- Create kinect reference frame -->
     <!-- Add mesh for kinect -->
@@ -41,5 +41,5 @@
       <collision>
         <geometry>
-          <box size="0.07 0.3 0.09"/>
+          <box size="0.01 0.05 0.01"/>
         </geometry>
       </collision>

Commit message: for foothold planning(fix real-time)

File: simple_dog_simulation/simpledog/urdf/laikago/my_laika.xacro (robot description, xacro)
@@ -106,6 +106,7 @@
         </collision>
     </link>
-    <xacro:include filename="$(find simpledog)/urdf/front_kinect.urdf.xacro"/>
-    <xacro:include filename="$(find simpledog)/urdf/right_kinect.urdf.xacro"/>
+   <xacro:include filename="$(find simpledog)/urdf/front_kinect.urdf.xacro"/>
+   <xacro:include filename="$(find simpledog)/urdf/front_high_kinect.urdf.xacro"/>
+   <xacro:include filename="$(find simpledog)/urdf/right_kinect.urdf.xacro"/>
     <!--load kinect urdf-->
       <xacro:front_kinect_camera prefix="front_camera" robot_namespace="$(arg robot_namespace)"/>
@@ -116,5 +117,12 @@
       </joint>
     <!--load kinect urdf-->
-      <xacro:right_kinect_camera prefix="right_camera" robot_namespace="$(arg robot_namespace)"/>
+      <xacro:front_high_kinect_camera prefix="front_high_camera" robot_namespace="$(arg robot_namespace)"/>
+      <joint name="front_high_kinect_frame_joint" type="fixed">
+        <origin xyz="0.28 0 0.1" rpy="0 0.1 0" />
+        <parent link="base"/>
+        <child link="front_high_camera_link"/>
+      </joint>
+    <!--load kinect urdf-->
+     <xacro:right_kinect_camera prefix="right_camera" robot_namespace="$(arg robot_namespace)"/>
       <joint name="right_kinect_frame_joint" type="fixed">
         <origin xyz="-0.0 -0.07 0.0" rpy="0 0.8 -1.57" />
