Commit message: final commit for laikago

File: simple_dog_simulation/simpledog/urdf/front_kinect.urdf.xacro (robot description, xacro)
@@ -26,5 +26,5 @@
 -->
 <robot xmlns:xacro="http://ros.org/wiki/xacro" name="front_kinect_camera">
-  <xacro:macro name="front_kinect_camera" params="prefix:=front_camera robot_namespace:=/">
+  <xacro:macro name="front_kinect_camera" params="prefix:=camera robot_namespace:=/">
     <!-- Create kinect reference frame -->
     <!-- Add mesh for kinect -->

File: simple_dog_simulation/simpledog/urdf/laikago/my_laika.xacro (robot description, xacro)
@@ -107,22 +107,38 @@
     </link>
    <xacro:include filename="$(find simpledog)/urdf/front_kinect.urdf.xacro"/>
+   <xacro:include filename="$(find simpledog)/urdf/stereo.urdf.xacro"/>
    <xacro:include filename="$(find simpledog)/urdf/front_high_kinect.urdf.xacro"/>
    <xacro:include filename="$(find simpledog)/urdf/right_kinect.urdf.xacro"/>
+   <xacro:include filename="$(find simpledog)/urdf/rear_kinect.urdf.xacro"/>
+   <xacro:include filename="$(find simpledog)/urdf/left_kinect.urdf.xacro"/>
     <!--load kinect urdf-->
-      <xacro:front_kinect_camera prefix="front_camera" robot_namespace="$(arg robot_namespace)"/>
+<!--load stereo_camera for vins-->
+<!--    <xacro:stereo_camera prefix="camera" robot_namespace="$(arg robot_namespace)"/>
+    <joint name="stereo_frame_joint" type="fixed">
+      <origin xyz="0.28 0.0 0.0" rpy="0 0 0" />
+      <parent link="base"/>
+      <child link="camera_link"/>
+    </joint> -->
+      <xacro:front_kinect_camera prefix="camera" robot_namespace="$(arg robot_namespace)"/>
       <joint name="front_kinect_frame_joint" type="fixed">
-        <origin xyz="0.28 0 0.0" rpy="0 0.8 0" />
+        <origin xyz="0.30 0 0.0" rpy="0 0.8 0" />
         <parent link="base"/>
-        <child link="front_camera_link"/>
+        <child link="camera_link"/>
       </joint>
+   <!--   <xacro:rear_kinect_camera prefix="rear_camera" robot_namespace="$(arg robot_namespace)"/>
+      <joint name="rear_kinect_frame_joint" type="fixed">
+        <origin xyz="-0.28 0 0.0" rpy="0 0.8 3.14" />
+        <parent link="base"/>
+        <child link="rear_camera_link"/>
+      </joint> -->
     <!--load kinect urdf-->
-      <xacro:front_high_kinect_camera prefix="front_high_camera" robot_namespace="$(arg robot_namespace)"/>
+     <!-- <xacro:front_high_kinect_camera prefix="front_high_camera" robot_namespace="$(arg robot_namespace)"/>
       <joint name="front_high_kinect_frame_joint" type="fixed">
         <origin xyz="0.28 0 0.1" rpy="0 0.1 0" />
         <parent link="base"/>
         <child link="front_high_camera_link"/>
-      </joint>
+      </joint> -->
     <!--load kinect urdf-->
-     <xacro:right_kinect_camera prefix="right_camera" robot_namespace="$(arg robot_namespace)"/>
+    <!-- <xacro:right_kinect_camera prefix="right_camera" robot_namespace="$(arg robot_namespace)"/>
       <joint name="right_kinect_frame_joint" type="fixed">
         <origin xyz="-0.0 -0.07 0.0" rpy="0 0.8 -1.57" />
@@ -130,4 +146,14 @@
         <child link="right_camera_link"/>
       </joint>
+     <xacro:left_kinect_camera prefix="left_camera" robot_namespace="$(arg robot_namespace)"/>
+      <joint name="left_kinect_frame_joint" type="fixed">
+        <origin xyz="-0.0 0.07 0.0" rpy="0 0.8 1.57" />
+        <parent link="base"/>
+        <child link="left_camera_link"/>
+      </joint> -->
+    <xacro:include filename="$(find simpledog)/urdf/VLP-16.urdf.xacro"/>
+    <VLP-16 parent="base">
+        <origin xyz="0.0  0  0.11" rpy="0 0 0" />
+    </VLP-16>
     <xacro:leg name="LF" mirror="1" mirror_dae="true" front_hind="1" front_hind_dae="true">
         <origin rpy="0 0 0" xyz="${leg_offset_x} ${leg_offset_y} 0"/>
